File: PCB/Asus Qcode - 3X/Asus Qcode.kicad_pcb (KiCad board)
At the start: 2 copper layers, 121.9 x 49.5 mm, 22 parts, among them J1 COM_DEBUG, J2 Conn_01x03_Pin, J3 Conn_01x02_Pin, SW1 Recall Codes

Commit message: More PCB Tweaks
Parts:
- moved REF** 0.64 mm to (132.1, 15.2)
Changed lines of the file:
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@@
   )
   (footprint "MountingHole:MountingHole_2.2mm_M2_Pad" (layer "F.Cu")
-    (at 131.445 15.24)
+    (at 132.08 15.24)
     (descr "Mounting Hole 2.2mm, M2")
     (tags "mounting hole 2.2mm m2")
